File: kicad/theremin.kicad_pcb (KiCad board)
At the start: 2 copper layers, 98 x 56 mm, 41 parts, among them J1 Eurorack Mono Jack, J2 Aerial, SW1 SW_SPDT, U1 4069, U2 4069, U3 LM386, U4 LP2950-5.0_TO92

Commit message: Updating with new footprints and some tweaks
Parts:
- removed D3: 1N4001, Diode_THT:D_DO-35_SOD27_P7.62mm_Horizontal
- removed H2: MountingHole_Pad, MountingHole:MountingHole_3.2mm_M3_DIN965_Pad
- added D4: 1N4148, Diode_THT:D_DO-35_SOD27_P7.62mm_Horizontal, F.Cu at (70.1, 89.4)
- added J3: Expression Attachment, Connector_PinHeader_2.54mm:PinHeader_1x02_P2.54mm_Vertical, F.Cu at (93.7, 131.4)
- added R12: 270k, Resistor_THT:R_Axial_DIN0207_L6.3mm_D2.5mm_P10.16mm_Horizontal, F.Cu at (93.0, 123.5)
- BT1: footprint Connector_PinHeader_2.54mm:PinHeader_1x02_P2.54mm_Vertical -> Battery:BatteryHolder_Eagle_12BH611-GR
- C1, C12, C2, C3, C4, C5, C7: footprint Rumblesan_Standard_Parts:C_Rect_L7.0mm_W3.5mm_P5.00mm -> Capacitor_THT:C_Rect_L7.0mm_W3.5mm_P5.00mm
- C10, C11, C6, C8, C9: footprint Rumblesan_Standard_Parts:CP_Radial_D5.0mm_P2.00mm -> Capacitor_THT:CP_Radial_D5.0mm_P2.50mm
- H1: footprint MountingHole:MountingHole_3.2mm_M3_DIN965_Pad -> project-footprints:BCM_Logo_small_Copper_Pad_15mmx15mm
- LS1: footprint Connector_PinHeader_2.54mm:PinHeader_1x02_P2.54mm_Vertical -> project-footprints:Speaker_PUIAudio_AS04008MR-21-R
- R1, R10, R11, R2, R3, R4, R5, R6, R7, R8, R9: footprint Rumblesan_Standard_Parts:R_Axial_DIN0207_L6.3mm_D2.5mm_P10.16mm_Horizontal -> Resistor_THT:R_Axial_DIN0207_L6.3mm_D2.5mm_P10.16mm_Horizontal
- RV2: value 100k -> 25k; footprint Rumblesan_Standard_Parts:Potentiometer_Alpha_RD901F-40-00D_Single_Vertical -> Potentiometer_THT:Potentiometer_Alpha_RD901F-40-00D_Single_Vertical
- RV3: footprint Rumblesan_Standard_Parts:Potentiometer_Alpha_RD901F-40-00D_Single_Vertical -> Potentiometer_THT:Potentiometer_Alpha_RD901F-40-00D_Single_Vertical
- SW1: footprint Rumblesan_Standard_Parts:SW_SPDT_DailyWell_Sub_MiniToggle -> Button_Switch_THT:SW_CuK_OS102011MA1QN1_SPDT_Angled
- U1, U2: footprint Rumblesan_Standard_Parts:DIP-14_W7.62mm_Socket -> Package_DIP:DIP-14_W7.62mm_Socket_LongPads
- U3: footprint Rumblesan_Standard_Parts:DIP-8_W7.62mm_Socket -> Package_DIP:DIP-8_W7.62mm_Socket_LongPads
- moved REF** 94.5 mm to (166.9, 36.6)
- moved LS1 67.4 mm to (151.9, 140.2), turned to 0 degrees
- moved BT1 36.3 mm to (49.3, 105.4)
- moved SW1 25.1 mm to (29.7, 70.1), turned to -90 degrees
- moved H1 20.1 mm to (91.7, 93.2)
Connections:
- C1 pad 1: Net-(J2-Pin_1) -> Net-(C1-Pad1)
- C1 pad 2: Net-(C1-Pad2) -> Net-(J2-Pin_1)
- C11 pad 1: Net-(D3-K) -> Net-(#FLG01-pwr)
- R1 pad 1: Net-(J2-Pin_1) -> Net-(R1-Pad1)
- R1 pad 2: Net-(R1-Pad2) -> Net-(J2-Pin_1)
- R10 pad 1: Net-(D3-K) -> Net-(SW1-A)
- R10 pad 2: Net-(SW1-A) -> Net-(#FLG01-pwr)
- R11 pad 1: Net-(R11-Pad1) -> GND
- R11 pad 2: GND -> Net-(R11-Pad2)
- R2 pad 1: Net-(J2-Pin_1) -> Net-(R2-Pad1)
- R2 pad 2: Net-(R2-Pad2) -> Net-(J2-Pin_1)
- R3 pad 1: Net-(C2-Pad1) -> Net-(R3-Pad1)
- R3 pad 2: Net-(R3-Pad2) -> Net-(C2-Pad2)
- R5 pad 1: Net-(D1-K) -> GND
- R5 pad 2: GND -> Net-(D1-K)
- R6 pad 1: Net-(C4-Pad2) -> Net-(C3-Pad2)
- R6 pad 2: Net-(C3-Pad2) -> Net-(C4-Pad2)
- R7 pad 1: Net-(C5-Pad2) -> Net-(C4-Pad2)
- R7 pad 2: Net-(C4-Pad2) -> Net-(C5-Pad2)
- R8 pad 1: Net-(C5-Pad2) -> Net-(C5-Pad1)
- R8 pad 2: Net-(C5-Pad1) -> Net-(C5-Pad2)
- R9 pad 1: Net-(C7-Pad1) -> GND
- R9 pad 2: GND -> Net-(C7-Pad1)
- RV1 pad 1: Net-(C2-Pad1) -> Net-(C2-Pad2)
- RV1 pad 2: Net-(R4-Pad1) -> Net-(R4-Pad2)
- RV1 pad 3: Net-(R4-Pad1) -> Net-(R4-Pad2)
- RV3 pad 3: Net-(R11-Pad1) -> Net-(R11-Pad2)
- U1 pad 1: Net-(R1-Pad2) -> Net-(R1-Pad1)
- U1 pad 2: Net-(R2-Pad2) -> Net-(R2-Pad1)
- U1 pad 3: Net-(R2-Pad2) -> Net-(R2-Pad1)
- U1 pad 4: Net-(C1-Pad2) -> Net-(C1-Pad1)
- U1 pad 5: Net-(C1-Pad2) -> Net-(C1-Pad1)
- U2 pad 10: Net-(C2-Pad2) -> Net-(C2-Pad1)
- U2 pad 11: Net-(R4-Pad2) -> Net-(R4-Pad1)
- U2 pad 12: Net-(R4-Pad2) -> Net-(R4-Pad1)
- U2 pad 13: Net-(R3-Pad2) -> Net-(R3-Pad1)
- U2 pad 9: Net-(C2-Pad2) -> Net-(C2-Pad1)
- U4 pad 3: Net-(D3-K) -> Net-(#FLG01-pwr)
Routing:
- net (no net): track 0.00 -> 67.9 mm
- net Net-(#FLG02-pwr): track 41.2 -> 0.00 mm
- net Net-(D3-K): track 16.9 -> 0.00 mm
- net Net-(SW1-A): track 3.19 -> 16.9 mm
- net Net-(R2-Pad2): track 10.8 -> 0.00 mm
- net Net-(BT1-+): track 7.00 -> 0.00 mm
- net Net-(C1-Pad2): track 6.81 -> 0.00 mm
- net Net-(R1-Pad2): track 5.53 -> 0.00 mm
- net Net-(R11-Pad1): track 4.24 -> 0.00 mm
- net GND: track 0.00 -> 4.24 mm
- net Net-(R3-Pad2): track 3.47 -> 0.00 mm
